File: fidget/fidget.sch (EAGLE design)
At the start: 15 parts, among them J1 HC_SR04, J2 RASPBERRY_PI_3_MODEL_B, M1 LEFT_MOTOR, M2 RIGHT_MOTOR, M3 SERVO, Q1 PN2222A, Q2 PN2222A

Commit message: Name the robot: fidget
Connections:
- net 5V: now also J2.5V@2
Changed lines of the file:
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@@
 <part name="J2" library="SparkFun-Connectors" deviceset="RASPBERRYPI-40-PIN-GPIO" device="_PTH" value="RASPBERRY_PI_3_MODEL_B"/>
 <part name="B2" library="SparkFun-Boards" deviceset="SPARKFUN_LOGIC_LEVEL_CONVERTER" device="" value="LOGIC_LEVEL_CONVERTER"/>
+<part name="SUPPLY7" library="SparkFun-PowerSymbols" deviceset="5V" device=""/>
 </parts>
 <sheets>
@@
 <instance part="J2" gate="G$1" x="73.66" y="25.4" rot="R90"/>
 <instance part="B2" gate="G$1" x="78.74" y="68.58" rot="R90"/>
+<instance part="SUPPLY7" gate="G$1" x="33.02" y="12.7"/>
 </instances>
 <busses>
@@
 <wire x1="76.2" y1="93.98" x2="76.2" y2="83.82" width="0.1524" layer="91"/>
 </segment>
+<segment>
+<pinref part="SUPPLY7" gate="G$1" pin="5V"/>
+<wire x1="33.02" y1="12.7" x2="33.02" y2="7.62" width="0.1524" layer="91"/>
+<wire x1="33.02" y1="7.62" x2="48.26" y2="7.62" width="0.1524" layer="91"/>
+<pinref part="J2" gate="G$1" pin="5V@2"/>
+<wire x1="48.26" y1="7.62" x2="48.26" y2="10.16" width="0.1524" layer="91"/>
+</segment>
 </net>
 <net name="7" class="0">
@@
 <wire x1="76.2" y1="50.8" x2="76.2" y2="45.72" width="0.1524" layer="91"/>
 <wire x1="76.2" y1="45.72" x2="43.18" y2="45.72" width="0.1524" layer="91"/>
-<wire x1="43.18" y1="45.72" x2="43.18" y2="7.62" width="0.1524" layer="91"/>
-<wire x1="43.18" y1="7.62" x2="53.34" y2="7.62" width="0.1524" layer="91"/>
+<wire x1="43.18" y1="45.72" x2="43.18" y2="2.54" width="0.1524" layer="91"/>
+<wire x1="43.18" y1="2.54" x2="53.34" y2="2.54" width="0.1524" layer="91"/>
 <pinref part="J2" gate="G$1" pin="3.3V@1"/>
-<wire x1="53.34" y1="7.62" x2="53.34" y2="10.16" width="0.1524" layer="91"/>
-</segment>
-</net>
+<wire x1="53.34" y1="2.54" x2="53.34" y2="10.16" width="0.1524" layer="91"/>
+</segment>
+</net>
